Commit message: Included Isaac Sim USD for lab automation project

File: config/tm5-900.ros2_control.xacro (robot description, xacro)
@@ -1,52 +1,76 @@
 <?xml version="1.0"?>
 <robot xmlns:xacro="http://www.ros.org/wiki/xacro">
-    <xacro:macro name="tm5-900_ros2_control" params="name initial_positions_file">
+    <xacro:macro name="tm5-900_ros2_control" params="name initial_positions_file ros2_control_hardware_type">
         <xacro:property name="initial_positions" value="${xacro.load_yaml(initial_positions_file)['initial_positions']}"/>
         <ros2_control name="${name}" type="system">
             <hardware>
-                <!-- By default, set up controllers for simulation. This won't work on real hardware -->
-                <plugin>mock_components/GenericSystem</plugin>
+                <xacro:if value="${ros2_control_hardware_type == 'mock_components'}">
+                    <plugin>mock_components/GenericSystem</plugin>
+                </xacro:if>
+                <xacro:if value="${ros2_control_hardware_type == 'isaac'}">
+                    <plugin>topic_based_ros2_control/TopicBasedSystem</plugin>
+                    <param name="joint_commands_topic">/isaac_joint_commands</param>
+                    <param name="joint_states_topic">/joint_states</param>
+                </xacro:if>
             </hardware>
             <joint name="joint_1">
                 <command_interface name="position"/>
+                <command_interface name="velocity"/>
+                <command_interface name="effort"/>
                 <state_interface name="position">
                   <param name="initial_value">${initial_positions['joint_1']}</param>
                 </state_interface>
                 <state_interface name="velocity"/>
+                <state_interface name="effort"/>
             </joint>
             <joint name="joint_2">
                 <command_interface name="position"/>
+                <command_interface name="velocity"/>
+                <command_interface name="effort"/>
                 <state_interface name="position">
                   <param name="initial_value">${initial_positions['joint_2']}</param>
                 </state_interface>
                 <state_interface name="velocity"/>
+                <state_interface name="effort"/>
             </joint>
             <joint name="joint_3">
                 <command_interface name="position"/>
+                <command_interface name="velocity"/>
+                <command_interface name="effort"/>
                 <state_interface name="position">
                   <param name="initial_value">${initial_positions['joint_3']}</param>
                 </state_interface>
                 <state_interface name="velocity"/>
+                <state_interface name="effort"/>
             </joint>
             <joint name="joint_4">
                 <command_interface name="position"/>
+                <command_interface name="velocity"/>
+                <command_interface name="effort"/>
                 <state_interface name="position">
                   <param name="initial_value">${initial_positions['joint_4']}</param>
                 </state_interface>
                 <state_interface name="velocity"/>
+                <state_interface name="effort"/>
             </joint>
             <joint name="joint_5">
                 <command_interface name="position"/>
+                <command_interface name="velocity"/>
+                <command_interface name="effort"/>
                 <state_interface name="position">
                   <param name="initial_value">${initial_positions['joint_5']}</param>
                 </state_interface>
                 <state_interface name="velocity"/>
+                <state_interface name="effort"/>
             </joint>
             <joint name="joint_6">
                 <command_interface name="position"/>
+                <command_interface name="velocity"/>
+                <command_interface name="effort"/>
                 <state_interface name="position">
                   <param name="initial_value">${initial_positions['joint_6']}</param>
                 </state_interface>
                 <state_interface name="velocity"/>
+                <state_interface name="effort"/>
             </joint>
             <joint name="finger_joint">
@@ -56,4 +80,5 @@
                 </state_interface>
                 <state_interface name="velocity"/>
+                <state_interface name="effort"/>
             </joint>
         </ros2_control>

File: config/tm5-900.urdf.xacro (robot description, xacro)
@@ -2,10 +2,17 @@
 <robot xmlns:xacro="http://www.ros.org/wiki/xacro" name="tm5-900">
     <xacro:arg name="initial_positions_file" default="initial_positions.yaml" />
-    <!-- Import tm5-900_rg6 urdf file -->
+    <xacro:arg name="ros2_control_hardware_type" default="mock_components" />
+    <!-- Import tm5-900 urdf file -->
     <xacro:include filename="$(find tm_description)/xacro/tm5-900.urdf.xacro" />
+    <!-- Import RG6 gripper urdf file -->
     <xacro:include filename="$(find onrobot_rg_description)/urdf/onrobot_rg6_model_macro.xacro" />
-    <xacro:onrobot_rg6 prefix="" effector_base="flange"/>
+    <xacro:onrobot_rg6 prefix=""/>
     <!-- Import control_xacro -->
     <xacro:include filename="tm5-900.ros2_control.xacro" />
-    <xacro:tm5-900_ros2_control name="FakeSystem" initial_positions_file="$(arg initial_positions_file)"/>
+    <xacro:tm5-900_ros2_control name="FakeSystem" initial_positions_file="$(arg initial_positions_file)" ros2_control_hardware_type="$(arg ros2_control_hardware_type)"/>
+    <joint name="joint_tcp_fixed" type="fixed">
+        <parent link="flange"/>
+        <child link="base_link"/>
+        <origin rpy="0 0 1.57079632679" xyz="0 0.0 0.0"/>
+    </joint>
 </robot>
